File: Fuente de Poder.sch (KiCad schematic (older format))
At the start: 8 parts, among them J1 USB_B_Micro, U1 XR21B1411IL16TR-F, U2 MAX8887EZK33+

Commit message: Issue #1: Correción de las conexiones Bus
Connections:
- no-connect marks 0 -> 1
Other:
- note added: "NOTAS\n=======\n\n- IP4220CZ6 - Supresor de descargas electrostáticas (ESD) / Diodos TVS\n (agregar en revisión del diseño).\n- Pin LOWPOWER de chip UART está en modo "Higth power device" (ver datasheet).\n- Revisar conección VBUS_SENSE (ver datasheet).\n- El pin USB ID del conector se usa para funcionalidad OTG (sin conexión?).\n-"
- note removed: "NOTAS\n=======\n\n- IP4220CZ6 - Supresor de descargas electrostáticas (ESD) / Diodos TVS\n (agregar en revisión del diseño).\n- Pin LOWPOWER de chip UART está en modo "Higth power device" (ver datasheet).\n- Revisar conección VBUS_SENSE (ver datasheet).\n- El pin USB ID del conector se usa para funcionalidad OTG (sino se usa, a tierra).\n-"
Changed lines of the file:
@@
 Etapa reguladora de voltaje - +3V3
 Text Notes 750  7500 0    43   ~ 0
-NOTAS\n=======\n\n- IP4220CZ6 - Supresor de descargas electrostáticas (ESD) / Diodos TVS\n  (agregar en revisión del diseño).\n- Pin LOWPOWER de chip UART está en modo "Higth power device" (ver datasheet).\n- Revisar conección VBUS_SENSE (ver datasheet).\n- El pin USB ID del conector se usa para funcionalidad OTG (sino se usa, a tierra).\n-
+NOTAS\n=======\n\n- IP4220CZ6 - Supresor de descargas electrostáticas (ESD) / Diodos TVS\n  (agregar en revisión del diseño).\n- Pin LOWPOWER de chip UART está en modo "Higth power device" (ver datasheet).\n- Revisar conección VBUS_SENSE (ver datasheet).\n- El pin USB ID del conector se usa para funcionalidad OTG (sin conexión?).\n-
 Wire Wire Line
 	5750 1775 5275 1775
@@
 Text Notes 6350 5800 0    43   ~ 0
 Etapa USB-UART
+NoConn ~ 2800 2175
 $EndSCHEMATC

Commit message: Issue #1: Cambio de regulador de voltaje
Se reemplazó el MAX8887 de Maxim por el SP6260 de Maxlinear.
Parts:
- removed C3: 10n, symbol Device:C
- removed U2: MAX8887EZK33+, Mis Huellas:MAX8887EZK33, symbol MAX8887EZK33:MAX8887EZK33+
- added U2: SP6260GEK-L_TR, SOT-23-5, symbol SP6260GEKLTR:SP6260GEK-L_TR
- C2, C4: value 2.2u -> 1u
Connections:
- wire segments 35 -> 33
Changed lines of the file:
@@
 $EndDescr
-$Comp
-L MAX8887EZK33:MAX8887EZK33+ U2
-U 1 1 5F4D7F55
-P 5750 1775
-F 0 "U2" H 6550 2162 60  0000 C CNN
-F 1 "MAX8887EZK33+" H 6550 2056 60  0000 C CNN
-F 2 "Mis Huellas:MAX8887EZK33" H 6550 2015 60  0001 C CNN
-F 3 "https://datasheets.maximintegrated.com/en/ds/MAX8887-MAX8888.pdf" H 6575 2375 60  0000 C CNN
-	1    5750 1775
-	1    0    0    -1
-$EndComp
 $Comp
 L Device:C C2
@@
 P 5275 2000
 F 0 "C2" H 5390 2046 50  0000 L CNN
-F 1 "2.2u" H 5390 1955 50  0000 L CNN
+F 1 "1u" H 5390 1955 50  0000 L CNN
 F 2 "" H 5313 1850 50  0001 C CNN
 F 3 "~" H 5275 2000 50  0001 C CNN
@@
 P 7700 2000
 F 0 "C4" H 7815 2046 50  0000 L CNN
-F 1 "2.2u" H 7815 1955 50  0000 L CNN
+F 1 "1u" H 7815 1955 50  0000 L CNN
 F 2 "" H 7738 1850 50  0001 C CNN
 F 3 "~" H 7700 2000 50  0001 C CNN
@@
 $EndComp
 Wire Wire Line
-	5750 1875 5750 1775
-Connection ~ 5750 1775
-Wire Wire Line
 	5275 2250 5275 2150
 Wire Wire Line
@@
 Wire Wire Line
 	5275 1775 5275 1500
-$Comp
-L Device:C C3
-U 1 1 5F582968
-P 5750 2350
-F 0 "C3" H 5865 2396 50  0000 L CNN
-F 1 "10n" H 5865 2305 50  0000 L CNN
-F 2 "" H 5788 2200 50  0001 C CNN
-F 3 "~" H 5750 2350 50  0001 C CNN
-	1    5750 2350
-	1    0    0    -1
-$EndComp
-$Comp
-L power:GND #PWR010
-U 1 1 5F582972
-P 5750 2600
-F 0 "#PWR010" H 5750 2350 50  0001 C CNN
-F 1 "GND" H 5755 2427 50  0000 C CNN
-F 2 "" H 5750 2600 50  0001 C CNN
-F 3 "" H 5750 2600 50  0001 C CNN
-	1    5750 2600
-	1    0    0    -1
-$EndComp
-Wire Wire Line
-	5750 2600 5750 2500
-Wire Wire Line
-	5750 2075 5750 2200
 Wire Wire Line
 	7350 2575 7350 2175
@@
 NOTAS\n=======\n\n- IP4220CZ6 - Supresor de descargas electrostáticas (ESD) / Diodos TVS\n  (agregar en revisión del diseño).\n- Pin LOWPOWER de chip UART está en modo "Higth power device" (ver datasheet).\n- Revisar conección VBUS_SENSE (ver datasheet).\n- El pin USB ID del conector se usa para funcionalidad OTG (sin conexión?).\n-
 Wire Wire Line
-	5750 1775 5275 1775
-Wire Wire Line
 	2800 2075 3125 2075
 Wire Wire Line
@@
 F 1 "XR21B1411IL16TR-F" H 7225 4456 60  0000 C CNN
 F 2 "QFN-16" H 7225 4415 60  0001 C CNN
-F 3 "https://www.maxlinear.com/ds/xr21b1411.pdf" H 7250 4750 60  0000 C CNN
+F 3 "https://www.maxlinear.com/ds/xr21b1411.pdf" H 7250 4750 60  0001 C CNN
 	1    5625 4175
 	1    0    0    -1
@@
 Etapa USB-UART
 NoConn ~ 2800 2175
+$Comp
+L SP6260GEKLTR:SP6260GEK-L_TR U2
+U 1 1 5F5C0B18
+P 5750 1775
+F 0 "U2" H 6550 2162 60  0000 C CNN
+F 1 "SP6260GEK-L_TR" H 6550 2056 60  0000 C CNN
+F 2 "SOT-23-5" H 6550 2015 60  0001 C CNN
+F 3 "" H 5750 1775 60  0000 C CNN
+	1    5750 1775
+	1    0    0    -1
+$EndComp
+Wire Wire Line
+	5275 1775 5750 1775
+Wire Wire Line
+	5750 1875 5750 1775
+Connection ~ 5750 1775
 $EndSCHEMATC

Commit message: Issue #1: Incorporación de conector para debug
Se agrega el conector estandar para ARM de 10 pines para debug con SWD.
Como referencia use la nota de aplicación AN0002.1
Parts:
- renumbered C4 to C3
Changed lines of the file:
@@
 $EndComp
 $Comp
-L Device:C C4
+L Device:C C3
 U 1 1 5F57B99E
 P 7700 2000
-F 0 "C4" H 7815 2046 50  0000 L CNN
+F 0 "C3" H 7815 2046 50  0000 L CNN
 F 1 "1u" H 7815 1955 50  0000 L CNN
 F 2 "" H 7738 1850 50  0001 C CNN
@@
 $EndComp
 $Comp
-L power:GND #PWR011
+L power:GND #PWR010
 U 1 1 5F57C7C8
 P 7350 2575
-F 0 "#PWR011" H 7350 2325 50  0001 C CNN
+F 0 "#PWR010" H 7350 2325 50  0001 C CNN
 F 1 "GND" H 7355 2402 50  0000 C CNN
 F 2 "" H 7350 2575 50  0001 C CNN
@@
 $EndComp
 $Comp
-L power:GND #PWR012
+L power:GND #PWR011
 U 1 1 5F57CA66
 P 7700 2225
-F 0 "#PWR012" H 7700 1975 50  0001 C CNN
+F 0 "#PWR011" H 7700 1975 50  0001 C CNN
 F 1 "GND" H 7705 2052 50  0000 C CNN
 F 2 "" H 7700 2225 50  0001 C CNN
@@
 	7700 1775 8025 1775
 $Comp
-L power:+3V3 #PWR013
+L power:+3V3 #PWR012
 U 1 1 5F58570D
 P 8025 1500
-F 0 "#PWR013" H 8025 1350 50  0001 C CNN
+F 0 "#PWR012" H 8025 1350 50  0001 C CNN
 F 1 "+3V3" H 8040 1673 50  0000 C CNN
 F 2 "" H 8025 1500 50  0001 C CNN
@@
 VBUS
 $Comp
-L power:GND #PWR014
+L power:GND #PWR013
 U 1 1 5F59930E
 P 8825 5650
-F 0 "#PWR014" H 8825 5400 50  0001 C CNN
+F 0 "#PWR013" H 8825 5400 50  0001 C CNN
 F 1 "GND" H 8830 5477 50  0000 C CNN
 F 2 "" H 8825 5650 50  0001 C CNN

Commit message: Issue #2: Primer acercamiento al diseño de la PCB
Se modificaron los conectores externos de los pines GPIOs (para no
exponer los que se conectan a los cristales) y se realizó la
distribución inicial de componentes en la placa (sin conectarlos)
Parts:
- C1: footprint (none) -> Capacitor_SMD:C_0603_1608Metric_Pad1.05x0.95mm_HandSolder
- C2, C3: footprint (none) -> Capacitor_THT:CP_Radial_D5.0mm_P2.50mm
- J1: footprint (none) -> Connector_USB:USB_Micro-B_Molex_47346-0001
- R1: footprint (none) -> Resistor_SMD:R_0603_1608Metric_Pad1.05x0.95mm_HandSolder
- U1: footprint QFN-16 -> Mis Huellas:XR21B1411IL16TR-F
- U2: footprint SOT-23-5 -> Mis Huellas:SP6260GEKLTR
Changed lines of the file:
@@
 F 0 "C2" H 5390 2046 50  0000 L CNN
 F 1 "1u" H 5390 1955 50  0000 L CNN
-F 2 "" H 5313 1850 50  0001 C CNN
+F 2 "Capacitor_THT:CP_Radial_D5.0mm_P2.50mm" H 5313 1850 50  0001 C CNN
 F 3 "~" H 5275 2000 50  0001 C CNN
 	1    5275 2000
@@
 F 0 "C3" H 7815 2046 50  0000 L CNN
 F 1 "1u" H 7815 1955 50  0000 L CNN
-F 2 "" H 7738 1850 50  0001 C CNN
+F 2 "Capacitor_THT:CP_Radial_D5.0mm_P2.50mm" H 7738 1850 50  0001 C CNN
 F 3 "~" H 7700 2000 50  0001 C CNN
 	1    7700 2000
@@
 F 0 "J1" H 2557 2442 50  0000 C CNN
 F 1 "USB_B_Micro" H 2557 2351 50  0000 C CNN
-F 2 "" H 2650 1925 50  0001 C CNN
+F 2 "Connector_USB:USB_Micro-B_Molex_47346-0001" H 2650 1925 50  0001 C CNN
 F 3 "~" H 2650 1925 50  0001 C CNN
 	1    2500 1975
@@
 F 0 "U1" H 7225 4562 60  0000 C CNN
 F 1 "XR21B1411IL16TR-F" H 7225 4456 60  0000 C CNN
-F 2 "QFN-16" H 7225 4415 60  0001 C CNN
+F 2 "Mis Huellas:XR21B1411IL16TR-F" H 7225 4415 60  0001 C CNN
 F 3 "https://www.maxlinear.com/ds/xr21b1411.pdf" H 7250 4750 60  0001 C CNN
 	1    5625 4175
@@
 F 0 "C1" H 4240 4471 50  0000 L CNN
 F 1 "100n" H 4240 4380 50  0000 L CNN
-F 2 "" H 4163 4275 50  0001 C CNN
+F 2 "Capacitor_SMD:C_0603_1608Metric_Pad1.05x0.95mm_HandSolder" H 4163 4275 50  0001 C CNN
 F 3 "~" H 4125 4425 50  0001 C CNN
 	1    4125 4425
@@
 F 0 "R1" H 5520 3896 50  0000 L CNN
 F 1 "10k" H 5520 3805 50  0000 L CNN
-F 2 "" V 5380 3850 50  0001 C CNN
+F 2 "Resistor_SMD:R_0603_1608Metric_Pad1.05x0.95mm_HandSolder" V 5380 3850 50  0001 C CNN
 F 3 "~" H 5450 3850 50  0001 C CNN
 	1    5450 3850
@@
 F 0 "U2" H 6550 2162 60  0000 C CNN
 F 1 "SP6260GEK-L_TR" H 6550 2056 60  0000 C CNN
-F 2 "SOT-23-5" H 6550 2015 60  0001 C CNN
+F 2 "Mis Huellas:SP6260GEKLTR" H 6550 2015 60  0001 C CNN
 F 3 "" H 5750 1775 60  0000 C CNN
 	1    5750 1775

Commit message: Issue #2: PCB lista para primera prueba de concepto
Parts:
- C1: footprint Capacitor_SMD:C_0603_1608Metric_Pad1.05x0.95mm_HandSolder -> Capacitor_SMD:C_1206_3216Metric_Pad1.42x1.75mm_HandSolder
- C2, C3: footprint Capacitor_THT:CP_Radial_D5.0mm_P2.50mm -> Capacitor_SMD:C_1206_3216Metric_Pad1.42x1.75mm_HandSolder
- R1: footprint Resistor_SMD:R_0603_1608Metric_Pad1.05x0.95mm_HandSolder -> Resistor_SMD:R_1206_3216Metric_Pad1.42x1.75mm_HandSolder
Connections:
- net GND: no longer J1.6 (Shield)
- net CD: no longer names the net of U1.7 (GPIO1/*CD)
- net DSR: no longer names the net of U1.6 (GPIO2/*DSR)
- net DTR: no longer names the net of U1.5 (GPIO3/*DTR)
- net RWK: no longer names the net of U1.8 (GPIO0/*RI/*RWK)
- no-connect marks 1 -> 6
Changed lines of the file:
@@
 $Descr A4 11693 8268
 encoding utf-8
-Sheet 2 4
+Sheet 3 4
 Title "Placa de Desarrollo EFM32 - MCU ARM"
 Date "2020-08-30"
@@
 F 0 "C2" H 5390 2046 50  0000 L CNN
 F 1 "1u" H 5390 1955 50  0000 L CNN
-F 2 "Capacitor_THT:CP_Radial_D5.0mm_P2.50mm" H 5313 1850 50  0001 C CNN
+F 2 "Capacitor_SMD:C_1206_3216Metric_Pad1.42x1.75mm_HandSolder" H 5313 1850 50  0001 C CNN
 F 3 "~" H 5275 2000 50  0001 C CNN
 	1    5275 2000
@@
 F 0 "C3" H 7815 2046 50  0000 L CNN
 F 1 "1u" H 7815 1955 50  0000 L CNN
-F 2 "Capacitor_THT:CP_Radial_D5.0mm_P2.50mm" H 7738 1850 50  0001 C CNN
+F 2 "Capacitor_SMD:C_1206_3216Metric_Pad1.42x1.75mm_HandSolder" H 7738 1850 50  0001 C CNN
 F 3 "~" H 7700 2000 50  0001 C CNN
 	1    7700 2000
@@
 Text Label 3125 1975 0    43   ~ 0
 USB_D+
-Wire Wire Line
-	2500 2475 2500 2625
-Connection ~ 2500 2475
-Wire Wire Line
-	2500 2375 2500 2475
-Wire Wire Line
-	2400 2475 2500 2475
-Wire Wire Line
-	2400 2375 2400 2475
 $Comp
 L power:GND #PWR01
@@
 F 0 "C1" H 4240 4471 50  0000 L CNN
 F 1 "100n" H 4240 4380 50  0000 L CNN
-F 2 "Capacitor_SMD:C_0603_1608Metric_Pad1.05x0.95mm_HandSolder" H 4163 4275 50  0001 C CNN
+F 2 "Capacitor_SMD:C_1206_3216Metric_Pad1.42x1.75mm_HandSolder" H 4163 4275 50  0001 C CNN
 F 3 "~" H 4125 4425 50  0001 C CNN
 	1    4125 4425
@@
 F 0 "R1" H 5520 3896 50  0000 L CNN
 F 1 "10k" H 5520 3805 50  0000 L CNN
-F 2 "Resistor_SMD:R_0603_1608Metric_Pad1.05x0.95mm_HandSolder" V 5380 3850 50  0001 C CNN
+F 2 "Resistor_SMD:R_1206_3216Metric_Pad1.42x1.75mm_HandSolder" V 5380 3850 50  0001 C CNN
 F 3 "~" H 5450 3850 50  0001 C CNN
 	1    5450 3850
@@
 Text HLabel 8825 4275 2    43   Output ~ 0
 TX
-Text HLabel 8825 4475 2    43   BiDi ~ 0
-RWK
-Text HLabel 8825 4575 2    43   BiDi ~ 0
-CD
-Text HLabel 8825 4675 2    43   BiDi ~ 0
-DSR
-Text HLabel 8825 4775 2    43   BiDi ~ 0
-DTR
 Text HLabel 8825 4875 2    43   BiDi ~ 0
 CTS
@@
 	5750 1875 5750 1775
 Connection ~ 5750 1775
+NoConn ~ 8825 4775
+NoConn ~ 8825 4675
+NoConn ~ 8825 4575
+NoConn ~ 8825 4475
+Wire Wire Line
+	2500 2375 2500 2625
+NoConn ~ 2400 2375
 $EndSCHEMATC
